File: BikeUSBv2/BikeUSBv2.kicad_pcb (KiCad board)
At the start: 2 copper layers, 43.6 x 25.5 mm, 52 parts, among them J1 TYPE-C-31-M-16, J2 Conn_01x02_Female, Q1 MMBT3906, SW1 SW_Push, SW2 SW_Push, U1 TPS63020DSJR, U2 ATtiny1616-M

Commit message: all parts selected
Parts:
- D1: value yellow -> XL-2012UOC
- D2: value green -> XL-2012UGC
- D3: value blue -> XL-2012UBC
- D9: value red -> XL-2012SURC
- SW1, SW2: value SW_Push -> 1TS002E-2500-2500-CT
Changed lines of the file:
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@@
     (descr "LED SMD 0805 (2012 Metric), square (rectangular) end terminal, IPC_7351 nominal, (Body size source: https://docs.google.com/spreadsheets/d/1BsfQQcO9C6DZCsRaXUlFlo91Tg2WpOkGARC1WS5S8t0/edit?usp=sharing), generated with kicad-footprint-generator")
     (tags "LED handsolder")
+    (property "LCSC" "C965817")
     (property "Sheetfile" "BikeUSBv2.kicad_sch")
     (property "Sheetname" "")
@@
         (effects (font (size 1 1) (thickness 0.15)))
     )
-    (fp_text value "blue" (at 0 1.65) (layer "F.Fab")
+    (fp_text value "XL-2012UBC" (at 0 1.65) (layer "F.Fab")
         (effects (font (size 1 1) (thickness 0.15)))
     )
@@
     (descr "LED SMD 0805 (2012 Metric), square (rectangular) end terminal, IPC_7351 nominal, (Body size source: https://docs.google.com/spreadsheets/d/1BsfQQcO9C6DZCsRaXUlFlo91Tg2WpOkGARC1WS5S8t0/edit?usp=sharing), generated with kicad-footprint-generator")
     (tags "LED handsolder")
+    (property "LCSC" "C965813")
     (property "Sheetfile" "BikeUSBv2.kicad_sch")
     (property "Sheetname" "")
@@
         (effects (font (size 1 1) (thickness 0.15)))
     )
-    (fp_text value "yellow" (at 0 1.65) (layer "F.Fab")
+    (fp_text value "XL-2012UOC" (at 0 1.65) (layer "F.Fab")
         (effects (font (size 1 1) (thickness 0.15)))
     )
@@
     (descr "https://www.mouser.com/ds/2/60/RS-282G05A-SM_RT-1159762.pdf")
     (tags "SPST button tactile switch")
+    (property "LCSC" "C329185")
     (property "Sheetfile" "BikeUSBv2.kicad_sch")
     (property "Sheetname" "")
@@
         (effects (font (size 1 1) (thickness 0.15)))
     )
-    (fp_text value "SW_Push" (at 0 3 90) (layer "F.Fab")
+    (fp_text value "1TS002E-2500-2500-CT" (at 0 3 90) (layer "F.Fab")
         (effects (font (size 1 1) (thickness 0.15)))
     )
@@
     (descr "LED SMD 0805 (2012 Metric), square (rectangular) end terminal, IPC_7351 nominal, (Body size source: https://docs.google.com/spreadsheets/d/1BsfQQcO9C6DZCsRaXUlFlo91Tg2WpOkGARC1WS5S8t0/edit?usp=sharing), generated with kicad-footprint-generator")
     (tags "LED handsolder")
+    (property "LCSC" "C965812")
     (property "Sheetfile" "BikeUSBv2.kicad_sch")
     (property "Sheetname" "")
@@
         (effects (font (size 1 1) (thickness 0.15)))
     )
-    (fp_text value "red" (at 0 1.65 90) (layer "F.Fab")
+    (fp_text value "XL-2012SURC" (at 0 1.65 90) (layer "F.Fab")
         (effects (font (size 1 1) (thickness 0.15)))
     )
@@
     (descr "LED SMD 0805 (2012 Metric), square (rectangular) end terminal, IPC_7351 nominal, (Body size source: https://docs.google.com/spreadsheets/d/1BsfQQcO9C6DZCsRaXUlFlo91Tg2WpOkGARC1WS5S8t0/edit?usp=sharing), generated with kicad-footprint-generator")
     (tags "LED handsolder")
+    (property "LCSC" "C965815")
     (property "Sheetfile" "BikeUSBv2.kicad_sch")
     (property "Sheetname" "")
@@
         (effects (font (size 1 1) (thickness 0.15)))
     )
-    (fp_text value "green" (at 0 1.65) (layer "F.Fab")
+    (fp_text value "XL-2012UGC" (at 0 1.65) (layer "F.Fab")
         (effects (font (size 1 1) (thickness 0.15)))
     )
@@
     (property "Sim.Device" "D")
     (property "Sim.Pins" "1=K 2=A")
+    (property "dnp" "")
+    (property "exclude_from_bom" "")
     (property "ki_description" "Schottky diode")
     (property "ki_keywords" "diode Schottky")
-    (attr smd exclude_from_pos_files)
+    (attr smd exclude_from_pos_files exclude_from_bom)
     (fp_text reference "D10" (at 0 -2 180) (layer "F.SilkS")
         (effects (font (size 1 1) (thickness 0.15)))
@@
     (descr "https://www.mouser.com/ds/2/60/RS-282G05A-SM_RT-1159762.pdf")
     (tags "SPST button tactile switch")
+    (property "LCSC" "C329185")
     (property "Sheetfile" "BikeUSBv2.kicad_sch")
     (property "Sheetname" "")
@@
         (effects (font (size 1 1) (thickness 0.15)))
     )
-    (fp_text value "SW_Push" (at 0 3 90) (layer "F.Fab")
-        (effects (font (size 1 1) (thickness 0.15)))
-    )
+    (fp_text value "1TS002E-2500-2500-CT" (at 0 3 90) (layer "F.Fab")
+        (effects (font (size 1 1) (thickness 0.15)))
+    )

Commit message: forgot to save PCB
Parts:
- J2: value Conn_01x02_Female -> JST S2B-EH(LF)(SN)
- SW1, SW2: value 1TS002E-2500-2500-CT -> 1TS002E-2500-2501-CT
Changed lines of the file:
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@@
     (descr "https://www.mouser.com/ds/2/60/RS-282G05A-SM_RT-1159762.pdf")
     (tags "SPST button tactile switch")
-    (property "LCSC" "C329185")
+    (property "LCSC" "C255802")
     (property "Sheetfile" "BikeUSBv2.kicad_sch")
     (property "Sheetname" "")
@@
         (effects (font (size 1 1) (thickness 0.15)))
     )
-    (fp_text value "1TS002E-2500-2500-CT" (at 0 3 90) (layer "F.Fab")
+    (fp_text value "1TS002E-2500-2501-CT" (at 0 3 90) (layer "F.Fab")
         (effects (font (size 1 1) (thickness 0.15)))
     )
@@
     (descr "https://www.mouser.com/ds/2/60/RS-282G05A-SM_RT-1159762.pdf")
     (tags "SPST button tactile switch")
-    (property "LCSC" "C329185")
+    (property "LCSC" "C255802")
     (property "Sheetfile" "BikeUSBv2.kicad_sch")
     (property "Sheetname" "")
@@
         (effects (font (size 1 1) (thickness 0.15)))
     )
-    (fp_text value "1TS002E-2500-2500-CT" (at 0 3 90) (layer "F.Fab")
+    (fp_text value "1TS002E-2500-2501-CT" (at 0 3 90) (layer "F.Fab")
         (effects (font (size 1 1) (thickness 0.15)))
     )
@@
     (descr "JST EH series connector, S2B-EH (http://www.jst-mfg.com/product/pdf/eng/eEH.pdf), generated with kicad-footprint-generator")
     (tags "connector JST EH horizontal")
+    (property "LCSC" "C514173")
     (property "Sheetfile" "BikeUSBv2.kicad_sch")
     (property "Sheetname" "")
@@
         (effects (font (size 1 1) (thickness 0.15)) (justify mirror))
     )
-    (fp_text value "Conn_01x02_Female" (at 1.25 -2.7 90) (layer "B.Fab")
+    (fp_text value "JST S2B-EH(LF)(SN)" (at 1.25 -2.7 90) (layer "B.Fab")
         (effects (font (size 1 1) (thickness 0.15)) (justify mirror))
     )

Commit message: smaller fixes
Routing:
- net +5V: track 63.4 -> 62.2 mm

Commit message: stuff
Parts:
- renumbered D9 to D4, D4 to D5, D5 to D6, D6 to D8, D8 to D9

Commit message: half capacitance, but cheaper
Parts:
- C9: value 1F -> 4700µF
